Commit message: Modify car apperance and footprint

File: src/simu/urdf/xju_model.gazebo.xacro (robot description, xacro)
@@ -5,4 +5,7 @@
   <gazebo reference="base_link">
     <material>Gazebo/Orange</material>
+  </gazebo>
+  <gazebo reference="pic_link">
+    <material>Gazebo/face</material>
   </gazebo>
   <gazebo reference="universal_wheel_link">

File: src/simu/urdf/xju_model.urdf.xacro (robot description, xacro)
@@ -42,4 +42,28 @@
     </collision>
   </link>
+  <!-- Picture -->
+  <link
+    name="pic_link">
+    <visual>
+      <origin
+        xyz="0 0 0"
+        rpy="0 0 0" />
+      <geometry>
+        <box size="0.4 0.39 0.001" />
+      </geometry>
+      <material name="orange" />
+    </visual>
+  </link>
+  <joint
+    name="joint_pic"
+    type="fixed">
+    <origin
+      xyz="0.1 0.0 0.5"
+      rpy="0 0 0" />
+    <parent
+      link="base_link" />
+    <child
+      link="pic_link" />
+  </joint>
   <!-- Wheel -->
   <link

Commit message: Add vlp16 & ultrasonic sensors

File: src/simu/urdf/xju_model.gazebo.xacro (robot description, xacro)
@@ -107,4 +107,46 @@
         <topicName>scan</topicName>
         <frameName>laser_link</frameName>
+      </plugin>
+    </sensor>
+  </gazebo>
+  <gazebo reference="top_laser_link">
+    <material>Gazebo/Red</material>
+    <sensor type="ray" name="$xju-VLP16">
+      <pose>0 0 0 0 0 0</pose>
+      <visualize>false</visualize>
+      <update_rate>10</update_rate>
+      <ray>
+        <scan>
+          <horizontal>
+            <samples>360</samples>
+            <resolution>1</resolution>
+            <min_angle>-3.141593</min_angle>
+            <max_angle>3.141593</max_angle>
+          </horizontal>
+          <vertical>
+            <samples>16</samples>
+            <resolution>1</resolution>
+            <min_angle>-0.261799</min_angle>
+            <max_angle>0.261799</max_angle>
+          </vertical>
+        </scan>
+        <range>
+          <min>0.01</min>
+          <max>30</max>
+          <resolution>0.01</resolution>
+        </range>
+        <noise>
+          <type>gaussian</type>
+          <mean>0.01</mean>
+          <stddev>0.0</stddev>
+        </noise>
+      </ray>
+      <plugin name="gazebo_ros_laser_controller" filename="libgazebo_ros_velodyne_laser.so">
+        <topicName>vlp_points</topicName>
+        <frameName>top_laser_link</frameName>
+        <organize_cloud>false</organize_cloud>
+        <min_range>0.01</min_range>
+        <max_range>30</max_range>
+        <gaussianNoise>0.01</gaussianNoise>
       </plugin>
     </sensor>
@@ -152,3 +194,155 @@
   </sensor>
  </gazebo>
+  <gazebo reference="ultra_left_front_link">
+     <material>Gazebo/Red</material>
+     <sensor type="ray" name="ultra_left_front">
+       <pose>0 0 0 0 0 0</pose>
+       <visualize>false</visualize>
+       <update_rate>10</update_rate>
+       <ray>
+         <scan>
+            <horizontal>
+               <samples>10</samples>
+               <resolution>1</resolution>
+               <min_angle>-0.1308</min_angle>
+               <max_angle>0.1308</max_angle>
+            </horizontal>
+            <vertical>
+               <samples>10</samples>
+               <resolution>1</resolution>
+               <min_angle>-0.1308</min_angle>
+               <max_angle>0.1308</max_angle>
+            </vertical>
+         </scan>
+         <range>
+            <min>0.02</min>
+            <max>1.5</max>
+            <resolution>0.02</resolution>
+         </range>
+       </ray>
+       <plugin name="gazebo_ros_range" filename="libgazebo_ros_range.so">
+         <gaussianNoise>0.005</gaussianNoise>
+         <alwaysOn>true</alwaysOn>
+         <updateRate>10</updateRate>
+         <topicName>/ultra_left_front</topicName>
+         <frameName>/ultra_left_front_link</frameName>
+         <fov>0.5</fov>
+         <radiation>ultrasound</radiation>
+       </plugin>
+     </sensor>
+  </gazebo>
+  <gazebo reference="ultra_left_back_link">
+     <material>Gazebo/Red</material>
+     <sensor type="ray" name="ultra_left_back">
+       <pose>0 0 0 0 0 0</pose>
+       <visualize>false</visualize>
+       <update_rate>10</update_rate>
+       <ray>
+         <scan>
+            <horizontal>
+               <samples>10</samples>
+               <resolution>1</resolution>
+               <min_angle>-0.1308</min_angle>
+               <max_angle>0.1308</max_angle>
+            </horizontal>
+            <vertical>
+               <samples>10</samples>
+               <resolution>1</resolution>
+               <min_angle>-0.1308</min_angle>
+               <max_angle>0.1308</max_angle>
+            </vertical>
+         </scan>
+         <range>
+            <min>0.02</min>
+            <max>1.5</max>
+            <resolution>0.02</resolution>
+         </range>
+       </ray>
+       <plugin name="gazebo_ros_range" filename="libgazebo_ros_range.so">
+         <gaussianNoise>0.005</gaussianNoise>
+         <alwaysOn>true</alwaysOn>
+         <updateRate>10</updateRate>
+         <topicName>/ultra_left_back</topicName>
+         <frameName>/ultra_left_back_link</frameName>
+         <fov>0.5</fov>
+         <radiation>ultrasound</radiation>
+       </plugin>
+     </sensor>
+  </gazebo>
+  <gazebo reference="ultra_right_back_link">
+     <material>Gazebo/Red</material>
+     <sensor type="ray" name="ultra_right_back">
+       <pose>0 0 0 0 0 0</pose>
+       <visualize>false</visualize>
+       <update_rate>10</update_rate>
+       <ray>
+         <scan>
+            <horizontal>
+               <samples>10</samples>
+               <resolution>1</resolution>
+               <min_angle>-0.1308</min_angle>
+               <max_angle>0.1308</max_angle>
+            </horizontal>
+            <vertical>
+               <samples>10</samples>
+               <resolution>1</resolution>
+               <min_angle>-0.1308</min_angle>
+               <max_angle>0.1308</max_angle>
+            </vertical>
+         </scan>
+         <range>
+            <min>0.02</min>
+            <max>1.5</max>
+            <resolution>0.02</resolution>
+         </range>
+       </ray>
+       <plugin name="gazebo_ros_range" filename="libgazebo_ros_range.so">
+         <gaussianNoise>0.005</gaussianNoise>
+         <alwaysOn>true</alwaysOn>
+         <updateRate>10</updateRate>
+         <topicName>/ultra_right_back</topicName>
+         <frameName>/ultra_right_back_link</frameName>
+         <fov>0.5</fov>
+         <radiation>ultrasound</radiation>
+       </plugin>
+     </sensor>
+  </gazebo>
+  <gazebo reference="ultra_right_front_link">
+     <material>Gazebo/Red</material>
+     <sensor type="ray" name="ultra_right_front">
+       <pose>0 0 0 0 0 0</pose>
+       <visualize>false</visualize>
+       <update_rate>10</update_rate>
+       <ray>
+         <scan>
+            <horizontal>
+               <samples>10</samples>
+               <resolution>1</resolution>
+               <min_angle>-0.1308</min_angle>
+               <max_angle>0.1308</max_angle>
+            </horizontal>
+            <vertical>
+               <samples>10</samples>
+               <resolution>1</resolution>
+               <min_angle>-0.1308</min_angle>
+               <max_angle>0.1308</max_angle>
+            </vertical>
+         </scan>
+         <range>
+            <min>0.02</min>
+            <max>1.5</max>
+            <resolution>0.02</resolution>
+         </range>
+       </ray>
+       <plugin name="gazebo_ros_range" filename="libgazebo_ros_range.so">
+         <gaussianNoise>0.005</gaussianNoise>
+         <alwaysOn>true</alwaysOn>
+         <updateRate>10</updateRate>
+         <topicName>/ultra_right_front</topicName>
+         <frameName>/ultra_right_front_link</frameName>
+         <fov>0.5</fov>
+         <radiation>ultrasound</radiation>
+       </plugin>
+     </sensor>
+  </gazebo>
 </robot>

File: src/simu/urdf/xju_model.urdf.xacro (robot description, xacro)
@@ -307,4 +307,39 @@
       k_velocity="0" />
   </joint>
+  <link name="top_laser_link">
+    <visual>
+      <origin
+        xyz="0 0 0"
+        rpy="0 0 0" />
+      <geometry>
+        <cylinder length="0.02" radius="0.01" />
+      </geometry>
+      <material name="red" />
+    </visual>
+    <visual>
+      <origin
+        xyz="0 0 -0.06"
+        rpy="0 0 0" />
+      <geometry>
+        <cylinder length="0.1" radius="0.0033" />
+      </geometry>
+      <material name="red" />
+    </visual>
+  </link>
+  <joint
+    name="joint_top_ladar"
+    type="fixed">
+    <origin
+      xyz="0.1 0 0.61"
+      rpy="0 0 0" />
+    <parent
+      link="base_link" />
+    <child
+      link="top_laser_link" />
+    <axis
+      xyz="0 0 0" />
+    <safety_controller
+      k_velocity="0" />
+  </joint>
   <!-- Camera -->
   <link name="camera_front_base">
@@ -332,3 +367,72 @@
     <child link="camera_front_link"/>
   </joint>
+  <!-- Ultrasonic -->
+    <link name="ultra_left_front_link">
+      <visual>
+        <origin
+          xyz="0 0 0"
+          rpy="0 0 0" />
+        <geometry>
+          <box size="0.01 0.01 0.01" />
+        </geometry>
+        <material name="red" />
+      </visual>
+    </link>
+    <joint name="ultra_left_front_joint" type="fixed">
+      <axis xyz="0 0 0" />
+      <origin xyz="0.3 0.195 0.1" rpy="0 0 0.7854"/>
+      <parent link="base_link"/>
+      <child link="ultra_left_front_link"/>
+    </joint>
+    <link name="ultra_left_back_link">
+      <visual>
+        <origin
+          xyz="0 0 0"
+          rpy="0 0 0" />
+        <geometry>
+          <box size="0.01 0.01 0.01" />
+        </geometry>
+        <material name="red" />
+      </visual>
+    </link>
+    <joint name="ultra_left_back_joint" type="fixed">
+      <axis xyz="0 0 0" />
+      <origin xyz="-0.1 0.195 0.1" rpy="0 0 2.3562"/>
+      <parent link="base_link"/>
+      <child link="ultra_left_back_link"/>
+    </joint>
+    <link name="ultra_right_back_link">
+      <visual>
+        <origin
+          xyz="0 0 0"
+          rpy="0 0 0" />
+        <geometry>
+          <box size="0.01 0.01 0.01" />
+        </geometry>
+        <material name="red" />
+      </visual>
+    </link>
+    <joint name="ultra_right_back_joint" type="fixed">
+      <axis xyz="0 0 0" />
+      <origin xyz="-0.1 -0.195 0.1" rpy="0 0 -2.3562"/>
+      <parent link="base_link"/>
+      <child link="ultra_right_back_link"/>
+    </joint>
+    <link name="ultra_right_front_link">
+      <visual>
+        <origin
+          xyz="0 0 0"
+          rpy="0 0 0" />
+        <geometry>
+          <box size="0.01 0.01 0.01" />
+        </geometry>
+        <material name="red" />
+      </visual>
+    </link>
+    <joint name="ultra_right_front_joint" type="fixed">
+      <axis xyz="0 0 0" />
+      <origin xyz="0.3 -0.195 0.1" rpy="0 0 -0.7854"/>
+      <parent link="base_link"/>
+      <child link="ultra_right_front_link"/>
+    </joint>
 </robot>

Commit message: Add QR code and modify camera config

File: src/simu/urdf/xju_model.gazebo.xacro (robot description, xacro)
@@ -155,15 +155,15 @@
     <material>Gazebo/Red</material>
   <sensor name="depth_camera_front" type="depth">
-    <update_rate>2</update_rate>
+    <update_rate>10</update_rate>
     <camera>
       <horizontal_fov>1.2386</horizontal_fov>
       <image>
-        <width>320</width>
-        <height>200</height>
+        <width>1280</width>
+        <height>720</height>
         <format>R8G8B8</format>
       </image>
       <clip>
-        <near>0.3</near>
-        <far>3</far>
+        <near>0.1</near>
+        <far>5</far>
       </clip>
     </camera>

File: src/simu/urdf/xju_model.urdf.xacro (robot description, xacro)
@@ -343,15 +343,5 @@
   </joint>
   <!-- Camera -->
-  <link name="camera_front_base">
-    <visual>
-      <origin
-        xyz="0 0 0"
-        rpy="0 0 0" />
-      <geometry>
-        <box size="0.01 0.04 0.01" />
-      </geometry>
-      <material name="red" />
-    </visual>
-  </link>
+  <link name="camera_front_base"/>
   <joint name="camera_front_base_joint" type="fixed">
     <axis xyz="0 0 0" />
