Commit message: Add tricycle model

File: src/simu/urdf/xju_tricycle_model.urdf.xacro (robot description, xacro)
@@ -3,5 +3,5 @@
   name="xju" xmlns:xacro="http://ros.org/wiki/xacro">
   <xacro:include filename="$(find xju_simu)/urdf/ackermann.xacro"/>
-  <xacro:include filename="$(find xju_simu)/urdf/xju_ackermann_model.gazebo.xacro"/>
+  <xacro:include filename="$(find xju_simu)/urdf/xju_tricycle_model.gazebo.xacro"/>
   <xacro:include filename="$(find xju_simu)/urdf/common_properties.xacro"/>
   <!-- Body -->
@@ -24,8 +24,8 @@
     <visual>
       <origin
-        xyz="0.13 0 0.05"
-        rpy="0 0 0" />
-      <geometry>
-        <box size="0.4 0.3 0.1" />
+        xyz="0.095 0 0.05"
+        rpy="0 0 0" />
+      <geometry>
+        <box size="0.33 0.3 0.1" />
       </geometry>
       <material name="orange" />
@@ -33,8 +33,8 @@
     <collision>
       <origin
-        xyz="0.13 0 0.05"
-        rpy="0 0 0" />
-      <geometry>
-        <box size="0.4 0.2 0.1" />
+        xyz="0.06 0 0.05"
+        rpy="0 0 0" />
+      <geometry>
+        <box size="0.26 0.2 0.1" />
       </geometry>
     </collision>
@@ -48,5 +48,5 @@
         rpy="0 0 0" />
       <geometry>
-        <box size="0.4 0.3 0.001" />
+        <box size="0.33 0.3 0.001" />
       </geometry>
       <material name="orange" />
@@ -57,5 +57,5 @@
     type="fixed">
     <origin
-      xyz="0.13 0.0 0.1"
+      xyz="0.095 0.0 0.1"
       rpy="0 0 0" />
     <parent
@@ -65,5 +65,5 @@
   </joint>
   <!-- Wheel -->
-  <link name="left_steering_hinge">
+  <link name="front_steering_hinge">
     <inertial>
       <origin xyz="0 0 0" rpy="0 0 0" />
@@ -85,13 +85,13 @@
     </collision>
   </link>
-  <joint name="left_steering_hinge_joint" type="revolute">
-    <origin xyz="0.26 0.125 0" rpy="0 0 0" />
+  <joint name="front_steering_hinge_joint" type="revolute">
+    <origin xyz="0.26 0 0" rpy="0 0 0" />
     <parent link="base_link" />
-    <child link="left_steering_hinge" />
+    <child link="front_steering_hinge" />
     <axis xyz="0 0 1" />
     <limit lower="-0.6" upper="0.6" effort="5.0" velocity="1000.0"/>
   </joint>
-  <xacro:steering_hinge_transmission name="left_steering_hinge" />
-  <link name="left_front_wheel">
+  <xacro:steering_hinge_transmission name="front_steering_hinge" />
+  <link name="front_wheel">
     <inertial>
       <origin xyz="0 0 0" rpy="0 0 0" />
@@ -113,68 +113,12 @@
     </collision>
   </link>
-  <joint name="left_front_wheel_joint" type="continuous">
-    <origin xyz="0 0.05 0" rpy="0 0 0" />
-    <parent link="left_steering_hinge" />
-    <child link="left_front_wheel" />
+  <joint name="front_wheel_joint" type="continuous">
+    <origin xyz="0 0 0" rpy="0 0 0" />
+    <parent link="front_steering_hinge" />
+    <child link="front_wheel" />
     <axis xyz="0 1 0" />
-    <limit effort="0" velocity="1000" />
-  </joint>
-  <xacro:wheel_transmission name="left_front_wheel" />
-  <link name="right_steering_hinge">
-    <inertial>
-      <origin xyz="0 0 0" rpy="0 0 0" />
-      <mass value="0.5" />
-      <inertia ixx="1.35E-05" ixy="0" ixz="0" iyy="2.5E-05" iyz="0" izz="1.35E-05" />
-    </inertial>
-    <visual>
-      <origin xyz="0 0 0" rpy="1.57 0 0" />
-      <geometry>
-        <cylinder length="0.01" radius="0.005" />
-      </geometry>
-      <material name="black" />
-    </visual>
-    <collision>
-      <origin xyz="0 0 0" rpy="1.57 0 0" />
-      <geometry>
-        <cylinder length="0.01" radius="0.005" />
-      </geometry>
-    </collision>
-  </link>
-  <joint name="right_steering_hinge_joint" type="revolute">
-    <origin xyz="0.26 -0.125 0" rpy="0 0 0" />
-    <parent link="base_link" />
-    <child link="right_steering_hinge" />
-    <axis xyz="0 0 1" />
-    <limit lower="-0.6" upper="0.6" effort="5.0" velocity="1000.0"/>
-  </joint>
-  <xacro:steering_hinge_transmission name="right_steering_hinge" />
-  <link name="right_front_wheel">
-    <inertial>
-      <origin xyz="0 0 0" rpy="0 0 0" />
-      <mass value="2" />
-      <inertia ixx="0.002867" ixy="0" ixz="0" iyy="0.0049" iyz="0" izz="0.002867" />
-    </inertial>
-    <visual>
-      <origin xyz="0 0 0" rpy="1.57 0 0" />
-      <geometry>
-        <cylinder length="0.05" radius="0.07" />
-      </geometry>
-      <material name="black" />
-    </visual>
-    <collision>
-      <origin xyz="0 0 0" rpy="1.57 0 0" />
-      <geometry>
-        <cylinder length="0.05" radius="0.07" />
-      </geometry>
-    </collision>
-  </link>
-  <joint name="right_front_wheel_joint" type="continuous">
-    <origin xyz="0 -0.05 0" rpy="0 0 0" />
-    <parent link="right_steering_hinge" />
-    <child link="right_front_wheel" />
-    <axis xyz="0 1 0" />
-    <limit effort="0" velocity="1000" />
-  </joint>
-  <xacro:wheel_transmission name="right_front_wheel" />
+    <limit effort="10" velocity="1000" />
+  </joint>
+  <xacro:wheel_transmission name="front_wheel" />
   <link name="left_rear_wheel">
     <inertial>
@@ -202,5 +146,5 @@
     <child link="left_rear_wheel" />
     <axis xyz="0 1 0" />
-    <limit effort="10" velocity="1000" />
+    <limit effort="0" velocity="1000" />
   </joint>
   <xacro:wheel_transmission name="left_rear_wheel" />
@@ -230,5 +174,5 @@
     <child link="right_rear_wheel" />
     <axis xyz="0 1 0" />
-    <limit effort="10" velocity="1000" />
+    <limit effort="0" velocity="1000" />
   </joint>
   <xacro:wheel_transmission name="right_rear_wheel" />
@@ -251,5 +195,5 @@
   </joint>
   <!-- Lidar -->
-  <link name="laser_link">
+  <link name="top_laser_link">
     <visual>
       <origin
@@ -263,8 +207,8 @@
     <visual>
       <origin
-        xyz="0 0 -0.06"
-        rpy="0 0 0" />
-      <geometry>
-        <cylinder length="0.1" radius="0.0033" />
+        xyz="0 0 -0.3"
+        rpy="0 0 0" />
+      <geometry>
+        <cylinder length="0.6" radius="0.0033" />
       </geometry>
       <material name="red" />
@@ -272,13 +216,13 @@
   </link>
   <joint
-    name="joint_ladar"
+    name="joint_top_ladar"
     type="fixed">
     <origin
-      xyz="0.13 0 0.21"
+      xyz="0.13 0 0.61"
       rpy="0 0 0" />
     <parent
       link="base_link" />
     <child
-      link="laser_link" />
+      link="top_laser_link" />
     <axis
       xyz="0 0 0" />
