Commit message: feat: support cartographer pure localization mode

File: src/simu/urdf/xju_model.urdf.xacro (robot description, xacro)
@@ -42,5 +42,5 @@
     </collision>
   </link>
-  <!-- Picture -->
+  <!-- Picture
   <link
     name="pic_link">
@@ -65,5 +65,5 @@
     <child
       link="pic_link" />
-  </joint>
+  </joint>-->
   <!-- Wheel -->
   <link
